Commit message: fix(viz): ground drone on launch pad, ground gate footers, and optimize color palette contrast
- Initialize drone directly on ground launch pad by default (initial_offset=None)
- Ground race gates firmly with upright posts, circular base plates, and ground threshold bars at Z=0
- Make drone front props opaque saturated cyan and rear props opaque saturated red (enlarged discs)
- Remap desired trajectory to Electric Neon Violet and actual flown trail to Vivid Hot Pink / Magenta
- Reserve Cyan strictly for front drone orientation and White/Silver for launch pad ring
- Upgrade gate frames to light metallic aluminium for crisp contrast against dark floor
- Add automated unit test in test_arena_and_gates.py verifying ground start and gate footer grounding

File: assets/gates/lemniscate_gates.urdf (robot description, URDF)
Before this commit: robot lemniscate_gates, 5 links, 4 joints
Links:
- link gate_1: geometry visual box size=0.015 0.20 1.602; visual box size=0.015 0.20 1.602
- link gate_2: geometry visual box size=0.015 0.20 1.602; visual box size=0.015 0.20 1.602
- link gate_3: geometry visual box size=0.015 0.20 1.602; visual box size=0.015 0.20 1.602
- link gate_4: geometry visual box size=0.015 0.20 1.602; visual box size=0.015 0.20 1.602
