Commit message: feat(viz): realistic arena ground, 7-gate RATM racing passages, hexacopter UI, and FPV OSD

File: assets/hexacopter.urdf (robot description, URDF)
Before this commit: robot hexacopter, 9 links, 8 joints
Links:
- link arm_1: mass 0.001 -> 0.0001; geometry visual box size=0.015 0.015 0.008; visual box size=0.25 0.022 0.002
- link arm_2: mass 0.001 -> 0.0001; geometry visual box size=0.015 0.015 0.008; visual box size=0.25 0.022 0.002
- link arm_3: mass 0.001 -> 0.0001; geometry visual box size=0.015 0.015 0.008; visual box size=0.25 0.022 0.002
- link arm_4: mass 0.001 -> 0.0001; geometry visual box size=0.015 0.015 0.008; visual box size=0.25 0.022 0.002
- link arm_5: mass 0.001 -> 0.0001; geometry visual box size=0.015 0.015 0.008; visual box size=0.25 0.022 0.002
- link arm_6: mass 0.001 -> 0.0001; geometry visual box size=0.015 0.015 0.008; visual box size=0.25 0.022 0.002
- link base_link: mass 3.646 -> 3.646000; geometry collision cylinder length=0.08 radius=0.25; visual box size=0.028 0.028 0.028
- link gear_left: mass 0.001 -> 0.0001; geometry visual cylinder length=0.10 radius=0.005; visual cylinder length=0.10 radius=0.005
- link gear_right: mass 0.001 -> 0.0001; geometry visual cylinder length=0.10 radius=0.005; visual cylinder length=0.10 radius=0.005

Commit message: feat(viz): export figures as both PNG and PDF, make airframe solid and rotors transparent
- Generate both high-res PNG and publication-ready 300 DPI PDF for all simulation setup figure variants.
- Make the entire quadrotor airframe body, arms, motors, mounts, and landing gear 100% solid and opaque.
- Render the 6 aerodynamic rotor discs with true semi-transparency (alpha = 0.50), significantly more solid than the delicate trajectory line (alpha = 0.20).

File: assets/hexacopter.urdf (robot description, URDF)
Before this commit: robot hexacopter, 9 links, 8 joints
Links:
- link arm_1: geometry visual box size=0.25 0.022 0.002; visual cylinder length=0.010 radius=0.008
- link arm_2: geometry visual box size=0.25 0.022 0.002; visual cylinder length=0.010 radius=0.008
- link arm_3: geometry visual box size=0.25 0.022 0.002; visual cylinder length=0.010 radius=0.008
- link arm_4: geometry visual box size=0.25 0.022 0.002; visual cylinder length=0.010 radius=0.008
- link arm_5: geometry visual box size=0.25 0.022 0.002; visual cylinder length=0.010 radius=0.008
- link arm_6: geometry visual box size=0.25 0.022 0.002; visual cylinder length=0.010 radius=0.008
