Commit message: refactor project to nominal visual geometric control

File: assets/drone/cf2.urdf (robot description, URDF)
Before this commit: robot pybullet_drone, 5 links, 4 joints
Links:
- link base_link: geometry collision cylinder length=0.08 radius=0.25; visual mesh filename=C:/Users/g202404900/Desktop/visual-geo-ctrl/assets/drone/cf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 scale=3.5 3.5 3.5
